File: Velos_1/_autosave-Velos_1.kicad_pcb (KiCad board)
At the start: 2 copper layers, 104.3 x 59.6 mm, 28 parts, among them J1 conector_motor, J2 S_Bus, J3 llave_habilitacion, J4 parada_emergencia, J5 V_in +9VDC, J6 Control Driver, J7 potenciometro, K1 Relay_SPDT, Q1 BC548, Q2 BC548, Q3 BC548, Q4 BC548, Q5 BC548, U1 LM358, U2 L7805

Commit message: placa
Routing:
- net /Power_on_motor: track 52.9 -> 52.4 mm
Other:
- board size 104.3 x 59.6 mm -> 99.7 x 58.2 mm
