File: Velos_1/Velos_1.kicad_pcb (KiCad board)
At the start: 2 copper layers, 104.3 x 59.6 mm, 28 parts, among them J1 conector_motor, J2 S_Bus, J3 llave_habilitacion, J4 parada_emergencia, J5 V_in +9VDC, J6 Control Driver, J7 potenciometro, K1 Relay_SPDT, Q1 BC548, Q2 BC548, Q3 BC548, Q4 BC548, Q5 BC548, U1 LM358, U2 L7805

Commit message: placa final
Parts:
- added J8: Control Driver_backup, Connector_PinHeader_2.54mm:PinHeader_1x06_P2.54mm_Vertical, F.Cu at (154.2, 114.5)
- added J9: Conn_01x01_Pin, Connector_PinHeader_2.54mm:PinHeader_1x01_P2.54mm_Vertical, F.Cu at (161.3, 86.2)
- C1: value 100uF -> 22uF
- R4: value 47k -> 10k
Connections:
- A2 pad A0: unconnected-(A2-PadA0) -> A0
- A2 pad A1: unconnected-(A2-PadA1) -> A1
- A2 pad A2: unconnected-(A2-PadA2) -> A2
- A2 pad A3: unconnected-(A2-PadA3) -> A3
- A2 pad GND2: unconnected-(A2-GND-PadGND2) -> GND
Routing:
- net GND: track 364.3 -> 380.4 mm
- net +5V: track 294.7 -> 302.1 mm
- net A3: track 0.00 -> 5.09 mm
- net A2: track 0.00 -> 5.09 mm
- net A1: track 0.00 -> 5.09 mm
- net A0: track 0.00 -> 5.09 mm
Other:
- board outline removed
